File: HW/STM32-FC/io_RC_INPUT.kicad_sch (KiCad schematic)
At the start: 10 parts, among them J10 ZH 1.5mm 3P, J11 ZH 1.5mm 4P, J8 PWM_Conn_3x01, J9 PWM_Conn_3x01, Q2 S9013

Commit message: 2025.01.17 : PCB layout
Parts:
- removed D7: 1N4148, Diode_SMD:D_SOD-523, symbol Device:D_Small_Filled
- removed J8, J9: PWM_Conn_3x01, PWM_Connector:PWM_Conn_3x01, symbol PWM_Connector:PWM_Conn_3x01
- added J6: PWM_Conn_3x14, PWM_Connector:PWM_Conn_3x14, symbol PWM_Connector:PWM_Conn_3x14
- J7: renamed from J10; footprint Connector_JST:JST_ZH_S3B-ZR-SM4A-TF_1x03-1MP_P1.50mm_Horizontal -> JST_ZH:JST_ZH_S3B-ZR-SM4A-TF_1x03-1MP_P1.50mm_Horizontal
- J8: renamed from J11; footprint Connector_JST:JST_ZH_S4B-ZR-SM4A-TF_1x04-1MP_P1.50mm_Horizontal -> JST_ZH:JST_ZH_S4B-ZR-SM4A-TF_1x04-1MP_P1.50mm_Horizontal
- renumbered R21 to R19, R19 to R21, R18 to R22
Connections:
- net +5V: now also J6.16 (5V_RCIN), J6.17 (5V_RSSI)
- net GND: now also J6.18 (GND)
- net PPM_IN: now also J6.14 (RSSI)
- net RSSI_IN: now also J6.13 (RCIN)
- net UART1_RX: no longer J8.1 (Pin_1)
- net UART1_TX: now also J8.1 (Pin_1)
- new net +5V_PWM: J6.15 (5V_CH)
- new net AUX_CH1: J6.9 (AUX1)
- new net AUX_CH2: J6.10 (AUX2)
- new net AUX_CH3: J6.11 (AUX3)
- new net AUX_CH4: J6.12 (AUX4)
- new net MAIN_CH1: J6.1 (CH1)
- new net MAIN_CH2: J6.2 (CH2)
- new net MAIN_CH3: J6.3 (CH3)
- new net MAIN_CH4: J6.4 (CH4)
- new net MAIN_CH5: J6.5 (CH5)
- new net MAIN_CH6: J6.6 (CH6)
- new net MAIN_CH7: J6.7 (CH7)
- new net MAIN_CH8: J6.8 (CH8)
Other:
- note added: "AUX1 : PB7 : TIM4_CH1 AUX2 : PE11 : TIM1_CH2 AUX3 : PE13 : TIM1_CH3 AUX4 : PE14 : TIM1_CH4 RCIN : PD15 : TIM4_CH4 (PPM) RSSI_IN : PC0 : ADC"
- note added: "ZH 1.5mm 4P PA9 : UART1_TX (Half Duplex)"
- note removed: "2.54mm 3P PC0 : RSSI_IN"
- note removed: "AUX1 : PB7 : TIM4_CH1 AUX2 : PE11 : TIM1_CH2 AUX3 : PE13 : TIM1_CH3 AUX4 : PE14 : TIM1_CH4"
- note removed: "RSSI"
- note removed: "ZH 1.5mm 4P PA9 : UART1_TX PA10 : UART1_RX"
- moved on the sheet: J7, J8, Q2, R19, R20, R21, R22
