File: HW/STM32-FC/_autosave-io_RC_INPUT.kicad_sch (KiCad schematic)
At the start: 9 parts, among them J6 PWM_Conn_3x14, J7 ZH 1.5mm 3P, J8 ZH 1.5mm 4P, Q2 S9013

Commit message: 2025.02.11 PCB DONE! MEMO UPDATING
Other:
- note added: "AUX1 : PB0 : TIM3_CH3 PB7 : TIM4_CH1 AUX2 : PB1 : TIM3_CH4 PE11 : TIM1_CH2 AUX3 : PE13 : TIM1_CH3 AUX4 : PE14 : TIM1_CH4 RCIN : PPM/SBUS/SRXL2 RSSI_IN : PC1 : ADC123_IN11"
- note added: "MAIN 1 : PB7 : TIM4_CH1 PA0 : TIM5_CH1 MAIN 2 : PA1 : TIM5_CH2 MAIN 3 : PA2 : TIM5_CH3 MAIN 4 : PA3 : TIM5_CH4 MAIN 5 : PC6 : TIM3_CH1 MAIN 6 : PC7 : TIM3_CH2 MAIN 7 : MAIN 8 :"
- note removed: "AUX1 : PB7 : TIM4_CH1 AUX2 : PE11 : TIM1_CH2 AUX3 : PE13 : TIM1_CH3 AUX4 : PE14 : TIM1_CH4 RCIN : PPM/SBUS/SRXL2 RSSI_IN : PC1 : ADC123_IN11"
- note removed: "MAIN 1 : PA0 : TIM5_CH1 MAIN 2 : PA1 : TIM5_CH2 MAIN 3 : PA2 : TIM5_CH3 MAIN 4 : PA3 : TIM5_CH4 MAIN 5 : PC6 : TIM3_CH1 MAIN 6 : PC7 : TIM3_CH2 MAIN 7 : PB0 : TIM3_CH3 MAIN 8 : PB1 : TIM3_CH4"
Changed lines of the file:
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@@
 		)
 	)
-	(text "MAIN 1 : PA0 : TIM5_CH1\nMAIN 2 : PA1 : TIM5_CH2\nMAIN 3 : PA2 : TIM5_CH3\nMAIN 4 : PA3 : TIM5_CH4\nMAIN 5 : PC6 : TIM3_CH1\nMAIN 6 : PC7 : TIM3_CH2\nMAIN 7 : PB0 : TIM3_CH3\nMAIN 8 : PB1 : TIM3_CH4"
+	(text "MAIN 1 : PB7 : TIM4_CH1\nPA0 : TIM5_CH1\nMAIN 2 : PA1 : TIM5_CH2\nMAIN 3 : PA2 : TIM5_CH3\nMAIN 4 : PA3 : TIM5_CH4\nMAIN 5 : PC6 : TIM3_CH1\nMAIN 6 : PC7 : TIM3_CH2\nMAIN 7 : \nMAIN 8 : "
 		(exclude_from_sim no)
 		(at 23.8641 18.0091 0)
@@
 		)
 	)
-	(text "AUX1 : PB7 : TIM4_CH1\nAUX2 : PE11 : TIM1_CH2\nAUX3 : PE13 : TIM1_CH3\nAUX4 : PE14 : TIM1_CH4\n\nRCIN : PPM/SBUS/SRXL2\nRSSI_IN : PC1 : ADC123_IN11"
+	(text "AUX1 : PB0 : TIM3_CH3\nPB7 : TIM4_CH1\nAUX2 : PB1 : TIM3_CH4\nPE11 : TIM1_CH2\nAUX3 : PE13 : TIM1_CH3\nAUX4 : PE14 : TIM1_CH4\n\nRCIN : PPM/SBUS/SRXL2\nRSSI_IN : PC1 : ADC123_IN11"
 		(exclude_from_sim no)
 		(at 23.8641 35.7891 0)
