File: HW/STM32-FC/io_communication.kicad_sch (KiCad schematic)
At the start: 17 parts, among them J11 GH 1.25mm 6P, J12 GH 1.25mm 6P, J13 GH 1.25mm 4P, J14 GH 1.25mm 4P, J15 GH 1.25mm 4P, U10 ATA6561-GBQW, U11 ATA6561-GBQW

Commit message: 2025.02.06 PCB routing done v3
Parts:
- J11, J12: footprint JST_GH:JST_GH_BM06B-GHS-TBT_06 -> JST_GH:JST_GH_SM06B-GHS-TB_06x1.25mm_Angled; LCSC C189892 -> C19626244
- J13, J14, J15: footprint JST_GH:JST_GH_BM04B-GHS-TBT_04 -> JST_GH:JST_GH_SM04B-GHS-TB_04x1.25mm_Angled; LCSC C161692 -> C20584968
Connections:
- net +5V: now also J11.1 (Pin_1), J12.1 (Pin_1), J13.1 (Pin_1), J14.1 (Pin_1), J15.1 (Pin_1); no longer J11.6 (Pin_6), J12.6 (Pin_6), J13.4 (Pin_4), J14.4 (Pin_4), J15.4 (Pin_4)
- net CAN1_N: now also J14.3 (Pin_3); no longer J14.2 (Pin_2)
- net CAN1_P: now also J14.2 (Pin_2); no longer J14.3 (Pin_3)
- net CAN2_N: now also J15.3 (Pin_3); no longer J15.2 (Pin_2)
- net CAN2_P: now also J15.2 (Pin_2); no longer J15.3 (Pin_3)
- net GND: now also J11.6 (Pin_6), J12.6 (Pin_6), J13.4 (Pin_4), J14.4 (Pin_4), J15.4 (Pin_4); no longer J11.1 (Pin_1), J12.1 (Pin_1), J13.1 (Pin_1), J14.1 (Pin_1), J15.1 (Pin_1)
- net I2C_SCL: now also J13.2 (Pin_2); no longer J13.3 (Pin_3)
- net I2C_SDA: now also J13.3 (Pin_3); no longer J13.2 (Pin_2)
- net UART2_CTS: now also J11.4 (Pin_4); no longer J11.3 (Pin_3)
- net UART2_RTS: now also J11.5 (Pin_5); no longer J11.2 (Pin_2)
- net UART2_RX: now also J11.3 (Pin_3); no longer J11.4 (Pin_4)
- net UART2_TX: now also J11.2 (Pin_2); no longer J11.5 (Pin_5)
- net UART3_CTS: now also J12.4 (Pin_4); no longer J12.3 (Pin_3)
- net UART3_RTS: now also J12.5 (Pin_5); no longer J12.2 (Pin_2)
- net UART3_RX: now also J12.3 (Pin_3); no longer J12.4 (Pin_4)
- net UART3_TX: now also J12.2 (Pin_2); no longer J12.5 (Pin_5)

Commit message: 2025.02.07 USB C Conn change v1
Parts:
- C31, C32, C33, C34: LCSC C1581 -> C1525
- J11, J12: LCSC C19626244 -> C133065
- J13, J14, J15: LCSC C20584968 -> C189895
Changed lines of the file:
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@@
 			)
 		)
-		(property "LCSC" "C1581"
+		(property "LCSC" "C1525"
 			(at 149.8538 30.48 0)
 			(effects
@@
 			)
 		)
-		(property "LCSC" "C19626244 "
+		(property "LCSC" "C133065"
 			(at 71.12 33.02 0)
 			(effects
@@
 			)
 		)
-		(property "LCSC" "C1581"
+		(property "LCSC" "C1525"
 			(at 116.8462 69.85 0)
 			(effects
@@
 			)
 		)
-		(property "LCSC" "C20584968 "
+		(property "LCSC" "C189895"
 			(at 71.12 113.03 0)
 			(effects
@@
 			)
 		)
-		(property "LCSC" "C1581"
+		(property "LCSC" "C1525"
 			(at 149.8538 71.12 0)
 			(effects
@@
 			)
 		)
-		(property "LCSC" "C1581"
+		(property "LCSC" "C1525"
 			(at 116.8462 29.21 0)
 			(effects
@@
 			)
 		)
-		(property "LCSC" "C20584968 "
+		(property "LCSC" "C189895"
 			(at 170.18 76.2 0)
 			(effects
@@
 			)
 		)
-		(property "LCSC" "C19626244 "
+		(property "LCSC" "C133065"
 			(at 71.12 73.66 0)
 			(effects
@@
 			)
 		)
-		(property "LCSC" "C20584968 "
+		(property "LCSC" "C189895"
 			(at 170.18 35.56 0)
 			(effects

Commit message: 2025.02.11 PCB DONE! MEMO UPDATING
Other:
- note added: "GH 1.25mm 4P CAN1_STBY : PC4 CAN1_RX : PD0 CAN1_TX : PD1"
- note added: "GH 1.25mm 4P CAN2_STBY : PC5 CAN2_RX : PB6 CAN2_TX : PB12"
- note added: "GH 1.25mm 4P I2C_SCL : PB8 : I2C1_SCL I2C_SCL : PB9 : I2C1_SDA"
- note removed: "GH 1.25mm 4P PA8 : I2C3_SCL PC9 : I2C3_SDA"
- note removed: "GH 1.25mm 4P PC4 : CAN1_STBY PD0 : CAN1_RX PD1 : CAN1_TX"
- note removed: "GH 1.25mm 4P PC5 : CAN2_STBY PB6 : CAN2_RX PB12 : CAN2_TX"
Changed lines of the file:
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@@
 	(title_block
 		(title "Communication")
-		(date "2025-02-05")
+		(date "2025-02-08")
 		(rev "A")
 		(company "NARAE")
@@
 		)
 	)
-	(text "GH 1.25mm 4P\n\nPC5 : CAN2_STBY\nPB6 : CAN2_RX\nPB12 : CAN2_TX"
+	(text "GH 1.25mm 4P\n\nCAN2_STBY : PC5\nCAN2_RX : PB6\nCAN2_TX : PB12"
 		(exclude_from_sim no)
 		(at 89.916 58.674 0)
@@
 		)
 	)
-	(text "GH 1.25mm 4P\n\nPC4 : CAN1_STBY\nPD0 : CAN1_RX\nPD1 : CAN1_TX"
+	(text "GH 1.25mm 4P\n\nCAN1_STBY : PC4\nCAN1_RX : PD0\nCAN1_TX : PD1"
 		(exclude_from_sim no)
 		(at 89.916 18.034 0)
@@
 		)
 	)
-	(text "GH 1.25mm 4P\n\nPA8 : I2C3_SCL\nPC9 : I2C3_SDA"
+	(text "GH 1.25mm 4P\n\nI2C_SCL : PB8 : I2C1_SCL\nI2C_SCL : PB9 : I2C1_SDA"
 		(exclude_from_sim no)
 		(at 23.876 99.314 0)

Commit message: Test software v1
Parts:
- renumbered C31 to C32, C32 to C33, C33 to C34, C34 to C35, R29 to R30, R30 to R31, R31 to R32, R32 to R33, R33 to R34, R34 to R35
