File: HW/STM32-FC/usb.kicad_sch (KiCad schematic)
At the start: 33 parts, among them J2 USB_C_USB2.0_14P, J3 GH 1.25mm 6P, Q2 PMDPB30XN, Q3 PMDPB55XP, U2 USBLC6-2SC6, U3 TPS62840, U4 TPS62840, U5 TPS62840

Commit message: BMI323 Work in progress
Parts:
- removed C15: 4.7uF, Capacitor_SMD:C_0402_1005Metric, symbol Device:C_Small
- removed C18: 10uF, Capacitor_SMD:C_0402_1005Metric, symbol Device:C_Small
- removed L2: 2.2u, VLS201610ET-2R2M:VLS201610ET-2R2M, symbol Device:L_Iron_Small
- removed R21: 267k, Resistor_SMD:R_0402_1005Metric, symbol Device:R_Small_US
- removed U4: TPS62840, Package_BGA:Texas_DSBGA-6_0.855x1.255mm_Layout2x3_P0.4mm_LevelC, symbol TPS62840:TPS62840YBG
Connections:
- net +3.3VA is gone; now on net +3.3V: C19.1, L3.2, U5.A2 (VOS)
- net GNDA is gone; now on net GND: C19.2, R22.1
- net GND: no longer U2.2 (GND)
- net USB_CONN_D+: no longer U2.3 (I/O2)
- net USB_CONN_D-: no longer U2.1 (I/O1)
- net USB_D+: no longer U2.4 (I/O2)
- net USB_D-: no longer U2.6 (I/O1)
- net VBUS: no longer U2.5 (VBUS)
Other:
- note removed: "3.3V for RC with Power Gating"
