File: HW/STM32-FC/memory.kicad_sch (KiCad schematic)
At the start: 9 parts, among them J4 TF-06A, U6 W25X40CLUXIG

Commit message: BMI323 Work in progress
Parts:
- U6: footprint W25X40CLUX:USON_LUXIG TR_WIN-L -> W25X40CLUX:USON_LUXIG_TR_HandSolder
Changed lines of the file:
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@@
 	(title_block
 		(title "Memory")
-		(date "2025-06-19")
+		(date "2025-06-23")
 		(rev "A")
 		(company "NARAE")
@@
 	)
 	(symbol
-		(lib_name "GND_2")
 		(lib_id "power:GND")
 		(at 184.15 45.72 90)
@@
 	)
 	(symbol
-		(lib_name "GND_5")
 		(lib_id "power:GND")
 		(at 142.24 45.72 270)
@@
 			)
 		)
-		(property "Description" ""
+		(property "Description" "Unpolarized capacitor, small symbol"
 			(at 53.34 48.26 0)
 			(effects
@@
 			)
 		)
-		(property "Description" ""
+		(property "Description" "Unpolarized capacitor, small symbol"
 			(at 107.95 44.45 0)
 			(effects
@@
 			)
 		)
-		(property "Footprint" "W25X40CLUX:USON_LUXIG TR_WIN-L"
+		(property "Footprint" "W25X40CLUX:USON_LUXIG_TR_HandSolder"
 			(at 80.01 36.83 0)
 			(effects
@@
 			)
 		)
-		(property "Datasheet" "https://www.winbond.com/resource-files/W25X40CL_G%2020210505.pdf"
+		(property "Datasheet" "kicad-embed://w25x40cl_f 20140325.pdf"
 			(at 80.01 36.83 0)
 			(effects
@@
 	)
 	(symbol
-		(lib_name "+3.3V_4")
 		(lib_id "power:+3.3V")
 		(at 133.35 21.59 0)
